Commit message: add gripper tip joint and improve handling

File: piper/robot.urdf (robot description, URDF)
Before this commit: robot piper, 13 links, 12 joints
Links:
- added link gripper_end
Joints:
- added joint gripper_tip: type fixed, parent gripper_base, child gripper_end, origin xyz=0 0 0.138 rpy=0 0 0, axis 0 0 1
- joint gripper: limit lower=0 upper=0.1 effort=10 velocity=3 -> lower=0 upper=0.1 effort=10 velocity=1
- joint gripper_joint1: limit lower=0 upper=0.05 effort=10 velocity=3 -> lower=0 upper=0.05 effort=10 velocity=0.5
- joint gripper_joint2: limit lower=-0.05 upper=0 effort=10 velocity=3 -> lower=-0.05 upper=0 effort=10 velocity=0.5
- joint joint1: limit lower=-2.6179938 upper=2.6179938 effort=100 velocity=5 -> lower=-2.6179938 upper=2.6179938 effort=100 velocity=3
- joint joint2: limit lower=0 upper=3.1415926 effort=100 velocity=5 -> lower=0 upper=3.1415926 effort=100 velocity=3.4
- joint joint3: limit lower=-2.9670597 upper=0 effort=100 velocity=5 -> lower=-2.9670597 upper=0 effort=100 velocity=3.14
- joint joint4: limit lower=-1.7453292 upper=1.7453292 effort=100 velocity=5 -> lower=-1.7453292 upper=1.7453292 effort=100 velocity=3.92
- joint joint5: limit lower=-1.2217304 upper=1.2217304 effort=100 velocity=5 -> lower=-1.2217304 upper=1.2217304 effort=100 velocity=3.92
- joint joint6: limit lower=-2.0943951 upper=2.0943951 effort=100 velocity=5 -> lower=-2.0943951 upper=2.0943951 effort=100 velocity=3.92

Commit message: use placo's frame interpolation and improve readability

File: piper/robot.urdf (robot description, URDF)
Before this commit: robot piper, 14 links, 13 joints
Links:
- removed link gripper_end
- added link gripper_tcp_link
Joints:
- removed joint gripper_tip
- added joint gripper_tcp: type fixed, parent gripper_base, child gripper_tcp_link, origin xyz=0 0 0.138 rpy=0 0 0, axis 0 0 1

Commit message: use dynamic solver for better tracking & use joint regularization to avoid singularities

File: piper/robot.urdf (robot description, URDF)
Before this commit: robot piper, 14 links, 13 joints
Joints:
- joint gripper: limit lower=0 upper=0.1 effort=10 velocity=3 -> lower=0 upper=0.1 effort=10 velocity=1
- joint gripper_joint1: limit lower=0 upper=0.05 effort=10 velocity=3 -> lower=0 upper=0.05 effort=10 velocity=0.5
- joint gripper_joint2: limit lower=-0.05 upper=0 effort=10 velocity=3 -> lower=-0.05 upper=0 effort=10 velocity=0.5

Commit message: fix torque limits

File: piper/robot.urdf (robot description, URDF)
Before this commit: robot piper, 14 links, 13 joints
Joints:
- joint joint1: limit lower=-2.6179938 upper=2.6179938 effort=100 velocity=3 -> lower=-2.6179938 upper=2.6179938 effort=32 velocity=3
- joint joint2: limit lower=0 upper=3.1415926 effort=100 velocity=3 -> lower=0 upper=3.1415926 effort=32 velocity=3
- joint joint3: limit lower=-2.9670597 upper=0 effort=100 velocity=3 -> lower=-2.9670597 upper=0 effort=32 velocity=3
- joint joint4: limit lower=-1.7453292 upper=1.7453292 effort=100 velocity=3 -> lower=-1.7453292 upper=1.7453292 effort=6.5 velocity=3
- joint joint5: limit lower=-1.2217304 upper=1.2217304 effort=100 velocity=3 -> lower=-1.2217304 upper=1.2217304 effort=6.5 velocity=3
- joint joint6: limit lower=-2.0943951 upper=2.0943951 effort=100 velocity=3 -> lower=-2.0943951 upper=2.0943951 effort=6.5 velocity=3
